File: tinyFINITY.kicad_pcb (KiCad board)
At the start: 2 copper layers, 97 parts, among them U1 AP131-33, U3 2xSPDT, U4 STM32F058C8Ux, U5 LP2985AIM5-1.8/NOPB, X2 8MHz

Commit message: board outline
Parts:
- added D2: BAS70L, custom:SC75, F.Cu at (239.2, 94.6)
- added D3: BAS70L, custom:SC75, F.Cu at (241.7, 94.6)
- added H1: hole, custom:mouting_hole, F.Cu at (246.5, 125.8)
- added H2: hole, custom:mouting_hole, F.Cu at (247.9, 131.1)
- added H3: hole, custom:mouting_hole, F.Cu at (252.6, 126.1)
- added H4: hole, custom:mouting_hole, F.Cu at (250.1, 123.3)
- added R36: NC, custom:R_0402_CUSTOM, F.Cu at (246.9, 113.0)
- added R37: 75R, custom:R_0402_CUSTOM, F.Cu at (251.1, 110.6)
- added U2: RTC6705, custom:QFN40_6x6, F.Cu at (228.6, 130.2)
- added X1: 8MHZ 20pF 30ppm, custom:crystal_5032, F.Cu at (216.2, 97.2)
- U1: footprint TO_SOT_Packages_SMD:SOT-23-5 -> custom:SOT-23-5
- moved U3 246.2 mm to (234.9, 96.1)
- moved C25 238.7 mm to (240.1, 115.0)
- moved C26 237.3 mm to (246.6, 110.6)
- moved C8 236.5 mm to (241.3, 98.0)
- moved C2 236.4 mm to (242.3, 105.1)
- moved U1 236.3 mm to (234.1, 100.4)
- moved R4 236.3 mm to (251.4, 113.0)
- moved R14 234.7 mm to (248.9, 108.3)
- moved C1 234.6 mm to (250.9, 94.1)
- moved R6 234.5 mm to (250.9, 96.5)
- moved R26 234.0 mm to (237.9, 115.0)
- moved C4 233.3 mm to (246.4, 94.1)
- moved C17 233.3 mm to (237.8, 105.6)
- moved C29 232.7 mm to (248.6, 96.5)
- moved R15 232.0 mm to (246.8, 103.5)
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Connections:
- C16 pad 2: (no net) -> Net-(C16-Pad2)
- C18 pad 1: (no net) -> Net-(C18-Pad1)
- C19 pad 1: (no net) -> Net-(C19-Pad1)
- C20 pad 1: (no net) -> Net-(C20-Pad1)
- C5 pad 2: (no net) -> Net-(C5-Pad2)
- R10 pad 2: (no net) -> Net-(R10-Pad2)
- R32 pad 1: (no net) -> Net-(R32-Pad1)
- R4 pad 2: (no net) -> Net-(R4-Pad2)
- U3 pad 1: VIDEO_OVERLAY_WHITE -> VIDEO_OVERLAY_BLACK
- U3 pad 2: V_WHITE -> V_BLACK
- U3 pad 4: V_BLACK -> Net-(R37-Pad1)
- U3 pad 5: VIDEO_OVERLAY_BLACK -> Net-(D2-PadC)
- U3 pad 7: Net-(U3-Pad7) -> VIDEO
- U3 pad 9: Net-(U3-Pad7) -> V_WHITE
- U4 pad 41: VIDEO_OVERLAY_WHITE -> (no net)
Other:
- board outline added: 20 x 20 mm
- net class Default: clearance 0.2 -> 0.1524; trace_width 0.25 -> 0.1524; via_dia 0.8 -> 0.6858; via_drill 0.4 -> 0.3302
- rule pad_to_mask_clearance: 0.2 -> 0
- rule trace_clearance: 0.2 -> 0.1524
- rule trace_min: 0.2 -> 0.1524
- rule via_min_drill: 0.3 -> 0.3302
- rule via_min_size: 0.4 -> 0.6858
