File: tinyFINITY.kicad_pcb (KiCad board)
At the start: 2 copper layers, 20 x 20 mm, 102 parts, among them U1 AP131-33, U2 RTC6705, U3 ts3a44159, U4 STM32F301K8Ux, X1 8MHZ 20pF 30ppm, X2 8MHz, Y1 LF2012-A5R5AA

Commit message: cleanup
Parts:
- U1: footprint TO_SOT_Packages_SMD:SOT-23-5 -> custom:SOT-23-5

Commit message: footprint fix
Parts:
- C1: value 10nF -> 470pF
- C14, C15, C9: value 10pF HF -> '10pF
- C2: value 1uF -> 4.7uF
- C40: value 6.8pF HF -> '6.8pF
- C8: value 3.3pF HF -> '3.3pF
- L1, L2: value 1.2nH HF -> '1.2nH
- L3, L7: value 1nH HF -> '1nH
- L6: value 2.2nH HF -> '2.2nH
- R22: value 8R -> 1k37
- R24: value 4R -> 681
- R33: value 2R -> 348
- R34: value R -> 169
- U1: value AP131-33 -> MIC5205

Commit message: fixed L
Parts:
- L1, L2, L3, L4, L5, L6, L7: footprint custom:R_0402_CUSTOM -> custom:L_0402_CUSTOM

Commit message: backup
Parts:
- removed ANT1: 5400AT18A1000E, custom:CHIPANT_3216
- removed C40: '6.8pF, custom:C_0402_CUSTOM
- removed L6: '2.2nH, custom:L_0402_CUSTOM
- removed L7: '1nH, custom:L_0402_CUSTOM
- added C43: 10u 25V, custom:C_0805_CUSTOM, B.Cu at (233.6, 123.5)
- added C44: 680pF 50V, custom:C_0402_CUSTOM, F.Cu at (229.8, 124.4)
- added C45: 22uF, custom:C_0603_CUSTOM, B.Cu at (236.2, 127.2)
- added H1: hole, custom:mouting_hole, F.Cu at (237.2, 124.4)
- added H2: hole, custom:mouting_hole, F.Cu at (222.4, 128.9)
- added H3: hole, custom:mouting_hole, F.Cu at (221.2, 140.4)
- added H4: hole, custom:mouting_hole, F.Cu at (237.2, 140.4)
- added L8: 2.2uH, custom:L_SPM3012T, B.Cu at (233.8, 126.3)
- added R28: 100K, custom:R_0402_CUSTOM, F.Cu at (236.7, 128.2)
- added TP11: 5V, custom:TP_1.5x1.0, B.Cu at (238.0, 126.7)
- added TP12: ANT, custom:smd_1x1_round, F.Cu at (225.2, 123.4)
- added TP13: GND, custom:TP_1.5x1.0, B.Cu at (220.2, 130.2)
- added U5: TPS62153A-Q1, custom:VQFN16, B.Cu at (230.2, 126.0)
- C1, C2, C28, U1: moved to F.Cu
- moved C28 13.0 mm to (235.4, 126.7), turned to 90 degrees
- moved TP7 12.1 mm to (230.6, 123.2), turned to 180 degrees
- moved U1 11.2 mm to (233.0, 126.2), turned to 180 degrees
- moved C1 10.4 mm to (232.1, 123.9), turned to 180 degrees
- moved TP8 9.50 mm to (228.5, 123.2), turned to 180 degrees
- moved C2 7.39 mm to (230.5, 127.8), turned to 0 degrees
- moved C36 0.57 mm to (232.0, 133.5), turned to 180 degrees
Connections:
- C28 pad 1: VIN -> 5V
- U1 pad 1: VIN -> 5V
- U1 pad 3: VIN -> 5V
Routing:
- net GND: track 274.6 -> 321.4 mm, vias 71 -> 79
- net 5V: track 0.00 -> 20.0 mm, vias 0 -> 2
- net 3V3: track 84.6 -> 103.3 mm, vias 6 -> 5
- net VIN: track 6.40 -> 18.2 mm
- net Net-(L8-Pad1): track 0.00 -> 9.16 mm
- net Net-(R28-Pad1): track 0.00 -> 7.85 mm, vias 0 -> 1
- net Net-(C44-Pad2): track 0.00 -> 2.17 mm, vias 0 -> 1
- net Net-(C40-Pad1): track 2.15 -> 0.00 mm
- net Net-(TP12-Pad1): track 3.23 -> 1.50 mm
- net Net-(ANT1-Pad1): track 0.80 -> 0.00 mm
Other:
- board text added: "5V OUT"
- board text added: "GND"
- board text added: "rev 0.2 08/17"
- board text removed: "rev 0.1 05/17"

Commit message: multitabs
Parts:
- removed TP12: ANT, custom:smd_1x1_round
- added ANT1: COAX, custom:U.FL-R-SMT-1, B.Cu at (144.6, 97.3)
- added H3: hole, custom:mouting_hole, F.Cu at (153.1, 94.9)
- added H3: hole, custom:mouting_hole, F.Cu at (145.1, 94.9)
- added H3: hole, custom:mouting_hole, F.Cu at (143.9, 115.1)
- added H3: hole, custom:mouting_hole, F.Cu at (145.6, 115.1)
- added H3: hole, custom:mouting_hole, F.Cu at (144.4, 115.1)
- added H3: hole, custom:mouting_hole, F.Cu at (143.3, 115.1)
- added H3: hole, custom:mouting_hole, F.Cu at (145.0, 115.1)
- added H3: hole, custom:mouting_hole, F.Cu at (153.0, 115.1)
- added H3: hole, custom:mouting_hole, F.Cu at (151.3, 115.1)
- added H3: hole, custom:mouting_hole, F.Cu at (152.4, 115.1)
- added H3: hole, custom:mouting_hole, F.Cu at (153.6, 115.1)
- added H3: hole, custom:mouting_hole, F.Cu at (151.4, 94.9)
- added H3: hole, custom:mouting_hole, F.Cu at (151.9, 115.1)
- added H3: hole, custom:mouting_hole, F.Cu at (158.6, 101.5)
- added H3: hole, custom:mouting_hole, F.Cu at (158.6, 99.9)
- added H3: hole, custom:mouting_hole, F.Cu at (158.6, 101.0)
- added H3: hole, custom:mouting_hole, F.Cu at (158.6, 102.1)
- added H3: hole, custom:mouting_hole, F.Cu at (158.6, 100.5)
- added H3: hole, custom:mouting_hole, F.Cu at (158.6, 108.5)
- added H3: hole, custom:mouting_hole, F.Cu at (158.6, 110.1)
- added H3: hole, custom:mouting_hole, F.Cu at (158.6, 109.0)
- added H3: hole, custom:mouting_hole, F.Cu at (158.6, 107.9)
- added H3: hole, custom:mouting_hole, F.Cu at (152.5, 94.9)
- added H3: hole, custom:mouting_hole, F.Cu at (158.6, 109.5)
- added H3: hole, custom:mouting_hole, F.Cu at (138.4, 100.5)
- added H3: hole, custom:mouting_hole, F.Cu at (138.4, 102.1)
- added H3: hole, custom:mouting_hole, F.Cu at (138.4, 101.0)
- added H3: hole, custom:mouting_hole, F.Cu at (138.4, 99.9)
- added H3: hole, custom:mouting_hole, F.Cu at (138.4, 101.5)
- added H3: hole, custom:mouting_hole, F.Cu at (138.4, 109.5)
- added H3: hole, custom:mouting_hole, F.Cu at (138.4, 107.9)
- added H3: hole, custom:mouting_hole, F.Cu at (138.4, 109.0)
- added H3: hole, custom:mouting_hole, F.Cu at (138.4, 110.1)
- added H3: hole, custom:mouting_hole, F.Cu at (153.6, 94.9)
- added H3: hole, custom:mouting_hole, F.Cu at (138.4, 108.5)
- added H3: hole, custom:mouting_hole, F.Cu at (151.9, 94.9)
- added H3: hole, custom:mouting_hole, F.Cu at (143.9, 94.9)
- added H3: hole, custom:mouting_hole, F.Cu at (145.6, 94.9)
- added H3: hole, custom:mouting_hole, F.Cu at (144.5, 94.9)
- added H3: hole, custom:mouting_hole, F.Cu at (143.4, 94.9)
- added H4: hole, custom:mouting_hole, F.Cu at (134.3, 105.0)
- added H4: hole, custom:mouting_hole, F.Cu at (148.5, 90.8)
- added H4: hole, custom:mouting_hole, F.Cu at (162.6, 104.9)
- added H4: hole, custom:mouting_hole, F.Cu at (148.5, 119.2)
- moved H2 87.9 mm to (140.5, 97.0)
- moved C12 85.2 mm to (151.4, 109.2)
- moved C2 85.2 mm to (149.8, 100.4)
- moved C20 85.2 mm to (156.1, 102.3)
- moved C21 85.2 mm to (152.8, 113.8)
- moved C23 85.2 mm to (152.8, 103.7)
- moved C24 85.2 mm to (157.2, 105.8)
- moved C32 85.2 mm to (144.1, 111.9)
- moved C4 85.2 mm to (142.5, 103.3)
- moved C44 85.2 mm to (149.1, 97.0)
- moved D1 85.2 mm to (150.2, 114.0)
- moved R1 85.2 mm to (143.9, 102.8)
- moved R10 85.2 mm to (151.1, 105.6)
- moved R12 85.2 mm to (153.1, 105.0)
- moved R2 85.2 mm to (145.7, 112.8)
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Routing:
- net GND: track 321.4 -> 298.6 mm, vias 79 -> 76
- net Net-(ANT1-PadSIG): track 1.50 -> 1.18 mm, vias 0 -> 1
Other:
- board size 20 x 20 mm -> 36.6 x 36.6 mm
- board text added: "rev 0.3 08/17"
- board text removed: "rev 0.2 08/17"
